Commit message: updated params

File: unitree_ros-master/robots/aliengo_description/xacro/aliengo.urdf (robot description, URDF)
Before this commit: robot aliengo_description, 29 links, 28 joints
Joints:
- joint camera_joint: origin xyz=0.317 0 -0.032 rpy=0 0 0 -> xyz=0.3115 0 -0.032 rpy=0 0.1919 0
